Commit message: Setup initial scenario in .yaml

File: src/pick_and_place/exercise_1_tower_of_hanoi/description/tower_of_hanoi.urdf.xacro (robot description, xacro)
@@ -28,9 +28,10 @@
     <xacro:property name="initial_positions_file" default="$(arg initial_positions_file)"/>
     <link name="world" />
+    <xacro:property name="desk_number" value="1"/>
     <xacro:include filename="$(find rosiris_environment_description_common)/description/desk/desk_macro.xacro" />
     <xacro:desk
         prefix="$(arg prefix)"
         parent="world"
-        number="1"
+        number="${desk_number}"
         desk_height="0.8"
         desk_base_width="1"
@@ -38,4 +39,22 @@
         <origin xyz="1 1 0" rpy="0 0 0" />
     </xacro:desk>
+    <link name="$(arg prefix)desk_${desk_number}_place_location_left"/>
+    <joint name="$(arg prefix)desk_${desk_number}_place_location_left_joint" type="fixed">
+        <parent link="$(arg prefix)desk_${desk_number}_tabletop_link"/>
+        <child link="$(arg prefix)desk_${desk_number}_place_location_left"/>
+        <origin xyz="0.5 1.15 0.0" rpy="0 0 0" />
+    </joint>
+    <link name="$(arg prefix)desk_${desk_number}_place_location_middle"/>
+    <joint name="$(arg prefix)desk_${desk_number}_place_location_middle_joint" type="fixed">
+        <parent link="$(arg prefix)desk_${desk_number}_tabletop_link"/>
+        <child link="$(arg prefix)desk_${desk_number}_place_location_middle"/>
+        <origin xyz="0.5 0.8 0.0" rpy="0 0 0" />
+    </joint>
+    <link name="$(arg prefix)desk_${desk_number}_place_location_right"/>
+    <joint name="$(arg prefix)desk_${desk_number}_place_location_right_joint" type="fixed">
+        <parent link="$(arg prefix)desk_${desk_number}_tabletop_link"/>
+        <child link="$(arg prefix)desk_${desk_number}_place_location_right"/>
+        <origin xyz="0.5 0.45 0.0" rpy="0 0 0" />
+    </joint>
     <xacro:include filename="$(find rosiris_environment_description_common)/description/robot_mounts/simple_robot_mounts.xacro" />
     <xacro:cuboid_mount

Commit message: Add tip_frame and reference grapsframse on cubes

File: src/pick_and_place/exercise_1_tower_of_hanoi/description/tower_of_hanoi.urdf.xacro (robot description, xacro)
@@ -93,3 +93,9 @@
         <origin xyz="0 0 0" rpy="0 0 0" />  <!-- position robot relative to parent -->
     </xacro:load_robot>
+    <link name="robotiq_85_tip_link"/>
+    <joint name="robotiq_85_tip_link_joint" type="fixed">
+        <parent link="robotiq_85_base_link"/>
+        <child link="robotiq_85_tip_link"/>
+        <origin xyz="0 0 0.134722" rpy="0 0 0" />
+    </joint>
 </robot>
