Commit message: Define gripper as well

File: src/pick_and_place/pick_and_place_descriptions/robots/kortex/srdf/kortex_robot.srdf.xacro (robot description, xacro)
@@ -8,27 +8,27 @@
 <robot xmlns:xacro="http://wiki.ros.org/xacro">
     <xacro:macro name="kortex_robot" params="">
-        <!--GROUPS:
+        <!--GROUPS
         Representation of a set of joints and links. This can be useful for specifying DOF to plan
         for, defining arms, end effectors, etc-->
-        <!--LINKS:
+        <!--LINKS
         When a link is specified, the parent joint of that link (if it exists) is automatically
         included-->
-        <!--JOINTS:
+        <!--JOINTS
         When a joint is specified, the child link of that joint (which will always exist) is
         automatically included-->
-        <!--CHAINS:
+        <!--CHAINS
         When a chain is specified, all the links along the chain (including endpoints) are included
         in the group. Additionally, all the joints that are parents to included links are also
         included. This means that joints along the chain and the parent joint of the base link are
         included in the group-->
-        <!--SUBGROUPS:
+        <!--SUBGROUPS
         Groups can also be formed by referencing to already defined group names-->
-        <group name="kortex_eef">
-            <chain base_link="base_link" tip_link="kortex_eef" />
+        <group name="kortex_tool_group">
+            <chain base_link="base_link" tip_link="kortex_tool_link" />
         </group>
         <!--GROUP
-        STATES: Purpose: Define a named state for a particular group, in terms of joint values. This
+        STATES Purpose Define a named state for a particular group, in terms of joint values. This
         is useful to define states like 'folded arms'-->
-        <group_state name="Home" group="kortex_eef">
+        <group_state name="Home" group="kortex_tool_group">
             <joint name="joint_1" value="0" />
             <joint name="joint_2" value="0.26" />
@@ -39,5 +39,5 @@
             <joint name="joint_7" value="1.57" />
         </group_state>
-        <group_state name="Vertical" group="kortex_eef">
+        <group_state name="Vertical" group="kortex_tool_group">
             <joint name="joint_1" value="0" />
             <joint name="joint_2" value="0" />
@@ -48,9 +48,6 @@
             <joint name="joint_7" value="0" />
         </group_state>
-        <!--END
-        EFFECTOR: Purpose: Represent information about an end effector.-->
-        <end_effector name="kortex_eef" parent_link="kortex_eef" group="kortex_eef" />
         <!--DISABLE
-        COLLISIONS: By default it is assumed that any link of the robot could potentially come into
+        COLLISIONS By default it is assumed that any link of the robot could potentially come into
         collision with any other link in the robot. This tag disables collision checking between a
         specified pair of links. -->

File: src/pick_and_place/pick_and_place_descriptions/robots/kortex/urdf/load_kortex_robot.urdf.xacro (robot description, xacro)
@@ -20,5 +20,6 @@
             filename="$(find kortex_description)/arms/${arm}/${dof}dof/urdf/${arm}_macro.xacro" />
         <!-- Load the arm -->
-        <!-- Set some defaults for robot_ip, vision, gripper, gripper_joint_name which are not important-->
+        <!-- Set some defaults for robot_ip, vision, gripper, gripper_joint_name which are not
+        important-->
         <xacro:load_arm
             parent="${parent}"
@@ -41,9 +42,9 @@
         <!-- This is "universal" planning frame to which can be planned with an offset regardless of
         what tool might be attached -->
-        <link name="${prefix}kortex_eef" />
+        <link name="${prefix}kortex_tool_link" />
         <joint name="${prefix}tool_frame_joint" type="fixed">
             <origin xyz="0 0 0" rpy="0 0 0" />
             <parent link="${prefix}${last_arm_link}" />
-            <child link="${prefix}kortex_eef" />
+            <child link="${prefix}kortex_tool_link" />
             <axis xyz="0 0 0" />
         </joint>

File: src/pick_and_place/pick_and_place_descriptions/tower_of_hanoi/srdf/tower_of_hanoi.srdf.xacro (robot description, xacro)
@@ -1,8 +1,84 @@
 <?xml version="1.0" encoding="UTF-8"?>
 <robot xmlns:xacro="http://wiki.ros.org/xacro" name="tower_of_hanoi">
+    <!-- Inlcude the robot-->
     <xacro:include
         filename="$(find pick_and_place_descriptions)/robots/kortex/srdf/kortex_robot.srdf.xacro" />
     <xacro:kortex_robot />
-    <!-- Environment objects-->
+    <!-- Disable collision for robot mount point-->
     <disable_collisions link1="desk_1_link" link2="desk_1_cuboid_mount_link" reason="Adjacent" />
+    <!-- Inlcude the gripper-->
+    <xacro:include
+        filename="$(find pick_and_place_descriptions)/grippers/robotiq_2f_85/srdf/robotiq_2f_85_gripper.srdf.xacro" />
+    <xacro:robotiq_2f_85_gripper />
+    <group name="manipulator_robotiq_2f_85_tip">
+        <group name="kortex_tool_group"/>
+        <group name="robotiq_2f_85_gripper_tip"/>
+    </group>
+    <!--Disable
+    collisions between robot and gripper -->
+    <disable_collisions link1="bracelet_link" link2="robotiq_85_base_link" reason="Adjacent" />
+    <disable_collisions link1="bracelet_link" link2="robotiq_85_left_finger_link" reason="Never" />
+    <disable_collisions link1="bracelet_link" link2="robotiq_85_left_finger_tip_link" reason="Never" />
+    <disable_collisions link1="bracelet_link" link2="robotiq_85_left_inner_knuckle_link"
+        reason="Never" />
+    <disable_collisions link1="bracelet_link" link2="robotiq_85_left_knuckle_link" reason="Never" />
+    <disable_collisions link1="bracelet_link" link2="robotiq_85_right_finger_link" reason="Never" />
+    <disable_collisions link1="bracelet_link" link2="robotiq_85_right_finger_tip_link"
+        reason="Never" />
+    <disable_collisions link1="bracelet_link" link2="robotiq_85_right_inner_knuckle_link"
+        reason="Never" />
+    <disable_collisions link1="bracelet_link" link2="robotiq_85_right_knuckle_link" reason="Never" />
+    <disable_collisions link1="forearm_link" link2="robotiq_85_base_link" reason="Never" />
+    <disable_collisions link1="forearm_link" link2="robotiq_85_left_finger_link" reason="Never" />
+    <disable_collisions link1="forearm_link" link2="robotiq_85_left_finger_tip_link" reason="Never" />
+    <disable_collisions link1="forearm_link" link2="robotiq_85_left_inner_knuckle_link"
+        reason="Never" />
+    <disable_collisions link1="forearm_link" link2="robotiq_85_left_knuckle_link" reason="Never" />
+    <disable_collisions link1="forearm_link" link2="robotiq_85_right_finger_link" reason="Never" />
+    <disable_collisions link1="forearm_link" link2="robotiq_85_right_finger_tip_link" reason="Never" />
+    <disable_collisions link1="forearm_link" link2="robotiq_85_right_inner_knuckle_link"
+        reason="Never" />
+    <disable_collisions link1="forearm_link" link2="robotiq_85_right_knuckle_link" reason="Never" />
+    <disable_collisions link1="half_arm_2_link" link2="robotiq_85_left_finger_tip_link"
+        reason="Never" />
+    <disable_collisions link1="half_arm_2_link" link2="robotiq_85_left_inner_knuckle_link"
+        reason="Never" />
+    <disable_collisions link1="half_arm_2_link" link2="robotiq_85_right_finger_tip_link"
+        reason="Never" />
+    <disable_collisions link1="half_arm_2_link" link2="robotiq_85_right_inner_knuckle_link"
+        reason="Never" />
+    <disable_collisions link1="robotiq_85_base_link" link2="spherical_wrist_1_link" reason="Never" />
+    <disable_collisions link1="robotiq_85_base_link" link2="spherical_wrist_2_link" reason="Never" />
+    <disable_collisions link1="robotiq_85_left_finger_link" link2="spherical_wrist_1_link"
+        reason="Never" />
+    <disable_collisions link1="robotiq_85_left_finger_link" link2="spherical_wrist_2_link"
+        reason="Never" />
+    <disable_collisions link1="robotiq_85_left_finger_tip_link" link2="spherical_wrist_1_link"
+        reason="Never" />
+    <disable_collisions link1="robotiq_85_left_finger_tip_link" link2="spherical_wrist_2_link"
+        reason="Never" />
+    <disable_collisions link1="robotiq_85_left_inner_knuckle_link" link2="spherical_wrist_1_link"
+        reason="Never" />
+    <disable_collisions link1="robotiq_85_left_inner_knuckle_link" link2="spherical_wrist_2_link"
+        reason="Never" />
+    <disable_collisions link1="robotiq_85_left_knuckle_link" link2="spherical_wrist_1_link"
+        reason="Never" />
+    <disable_collisions link1="robotiq_85_left_knuckle_link" link2="spherical_wrist_2_link"
+        reason="Never" />
+    <disable_collisions link1="robotiq_85_right_finger_link" link2="spherical_wrist_1_link"
+        reason="Never" />
+    <disable_collisions link1="robotiq_85_right_finger_link" link2="spherical_wrist_2_link"
+        reason="Never" />
+    <disable_collisions link1="robotiq_85_right_finger_tip_link" link2="spherical_wrist_1_link"
+        reason="Never" />
+    <disable_collisions link1="robotiq_85_right_finger_tip_link" link2="spherical_wrist_2_link"
+        reason="Never" />
+    <disable_collisions link1="robotiq_85_right_inner_knuckle_link" link2="spherical_wrist_1_link"
+        reason="Never" />
+    <disable_collisions link1="robotiq_85_right_inner_knuckle_link" link2="spherical_wrist_2_link"
+        reason="Never" />
+    <disable_collisions link1="robotiq_85_right_knuckle_link" link2="spherical_wrist_1_link"
+        reason="Never" />
+    <disable_collisions link1="robotiq_85_right_knuckle_link" link2="spherical_wrist_2_link"
+        reason="Never" />
 </robot>

File: src/pick_and_place/pick_and_place_descriptions/tower_of_hanoi/urdf/tower_of_hanoi.urdf.xacro (robot description, xacro)
@@ -37,5 +37,25 @@
         <origin xyz="0 0.75 0" rpy="0 0 0" />
     </xacro:cuboid_mount>
-    <xacro:include filename="$(find pick_and_place_descriptions)/robots/kortex/urdf/load_kortex_robot.urdf.xacro" />
+    <!-- Place locations for the cubes-->
+    <link name="$(arg prefix)desk_${desk_number}_place_location_left" />
+    <joint name="$(arg prefix)desk_${desk_number}_place_location_left_joint" type="fixed">
+        <parent link="$(arg prefix)desk_${desk_number}_tabletop_link" />
+        <child link="$(arg prefix)desk_${desk_number}_place_location_left" />
+        <origin xyz="0.5 1.15 0.0" rpy="0 0 0" />
+    </joint>
+    <link name="$(arg prefix)desk_${desk_number}_place_location_middle" />
+    <joint name="$(arg prefix)desk_${desk_number}_place_location_middle_joint" type="fixed">
+        <parent link="$(arg prefix)desk_${desk_number}_tabletop_link" />
+        <child link="$(arg prefix)desk_${desk_number}_place_location_middle" />
+        <origin xyz="0.5 0.8 0.0" rpy="0 0 0" />
+    </joint>
+    <link name="$(arg prefix)desk_${desk_number}_place_location_right" />
+    <joint name="$(arg prefix)desk_${desk_number}_place_location_right_joint" type="fixed">
+        <parent link="$(arg prefix)desk_${desk_number}_tabletop_link" />
+        <child link="$(arg prefix)desk_${desk_number}_place_location_right" />
+        <origin xyz="0.5 0.45 0.0" rpy="0 0 0" />
+    </joint>
+    <xacro:include
+        filename="$(find pick_and_place_descriptions)/robots/kortex/urdf/load_kortex_robot.urdf.xacro" />
     <!-- initial position for simulations (Mock Hardware, Gazebo) -->
     <xacro:arg name="initial_positions_file"
@@ -55,4 +75,15 @@
         <origin xyz="0 0 0" rpy="0 0 0" />  <!-- position robot relative to parent -->
     </xacro:load_kortex_robot>
+    <xacro:include
+        filename="$(find pick_and_place_descriptions)/grippers/robotiq_2f_85/urdf/load_robotiq_2f_85_gripper.xacro" />
+    <xacro:load_robotiq_2f_85_gripper
+        parent="$(arg prefix)kortex_tool_link"
+        prefix="$(arg prefix)"
+        use_mock_hardware="$(arg use_mock_hardware)"
+        mock_sensor_commands="$(arg mock_sensor_commands)"
+        sim_gazebo="$(arg sim_gazebo)"
+        sim_isaac="$(arg sim_isaac)">
+        <origin xyz="0 0 0" rpy="0 0 0" />
+    </xacro:load_robotiq_2f_85_gripper>
     <xacro:if value="$(arg sim_gazebo)">
         <gazebo reference="$(arg world_link)">
